File: hbridge/hbridge.kicad_sch (KiCad schematic)
At the start: 12 parts, among them J1 MOSFET1, J2 MOSFET1, J3 MOSFET1, J4 MOSFET1, J5 Driver_in, J6 Driver_in, J7 Driver_in, J8 Driver_in, Q1 IRF3710, Q2 IRF3710, Q3 IRF3710, Q4 IRF3710

Commit message: Drivers added to half-bridge.
Parts:
- removed J1, J2, J3, J4: MOSFET1, TerminalBlock:TerminalBlock_Xinya_XY308-2.54-3P_1x03_P2.54mm_Horizontal, symbol Connector:Conn_01x03_Socket
- removed J5, J6, J7, J8: Driver_in, TerminalBlock:TerminalBlock_Xinya_XY308-2.54-6P_1x06_P2.54mm_Horizontal, symbol Connector:Conn_01x06_Socket
- removed Q1, Q2, Q3, Q4: IRF3710, Package_DirectFET:DirectFET_SQ, symbol Transistor_FET:IRF6713S
- added C1, C3: C, Capacitor_SMD:C_0805_2012Metric_Pad1.18x1.45mm_HandSolder, symbol Device:C
- added C2, C4, C5, C6: 0.47u, Capacitor_SMD:C_0805_2012Metric_Pad1.18x1.45mm_HandSolder, symbol Device:C
- added D10, D11, D13, D16: 1N4006, Diode_THT:D_DO-41_SOD81_P10.16mm_Horizontal, symbol Diode:1N4006
- added D12, D14, D15, D17, D18, D7, D8, D9: Green LED, LED_SMD:LED_1206_3216Metric_Pad1.42x1.75mm_HandSolder, symbol Device:LED
- added J1, J10, J4, J7: From_MCU, TerminalBlock:TerminalBlock_Xinya_XY308-2.54-6P_1x06_P2.54mm_Horizontal, symbol Connector_Generic:Conn_01x06
- added J11, J2, J5, J8: MOSFET_out, TerminalBlock:TerminalBlock_Xinya_XY308-2.54-3P_1x03_P2.54mm_Horizontal, symbol Connector_Generic:Conn_01x03
- added J12, J3, J6, J9: Conn_01x03, TerminalBlock:TerminalBlock_Xinya_XY308-2.54-3P_1x03_P2.54mm_Horizontal, symbol Connector_Generic:Conn_01x03
- added J13, J14: Conn_01x01_Socket, Connector_PinHeader_2.54mm:PinHeader_1x01_P2.54mm_Vertical, symbol Connector:Conn_01x01_Socket
- added J15, J16, J17, J18: VEE connector, Connector_PinHeader_2.54mm:PinHeader_1x03_P2.54mm_Vertical, symbol Connector:Conn_01x03_Socket
- added Q1, Q2, Q3, Q4: IRF3710, Package_TO_SOT_THT:TO-220-3_Vertical, symbol Transistor_FET:Q_Dual_NMOS_G1S2G2D2S1D1
- added R13, R14, R15, R22, R23, R24, R28, R29, R30, R34, R35, R36: 4.7k, Resistor_SMD:R_0805_2012Metric_Pad1.20x1.40mm_HandSolder, symbol Device:R
- added R16, R19, R25, R31: 550, Resistor_SMD:R_2512_6332Metric_Pad1.40x3.35mm_HandSolder, symbol Device:R
- added R17, R18, R20, R21, R26, R27, R32, R33: 10, Resistor_SMD:R_2512_6332Metric_Pad1.40x3.35mm_HandSolder, symbol Device:R
- added TP1, TP10, TP11, TP12, TP2, TP3, TP4, TP5, TP6, TP7, TP8, TP9: TestPoint, TestPoint:TestPoint_Loop_D2.50mm_Drill1.0mm, symbol Connector:TestPoint
- added U1: LDO-3.3, Package_TO_SOT_SMD:SOT-223-3_TabPin2, symbol Regulator_Linear:LT1963AxST-3.3
- added U5, U6, U7, U8: NSi6651A, Package_SO:SOIC-16W_7.5x10.3mm_P1.27mm, symbol Driver_FET:FAN7842
Connections:
- new net: D16.1 (K), R31.2
- new net: D16.2 (A), U8.2 (DESAT)
- new net: C3.1, J13.1 (Pin_1), U1.1 (IN)
- new net: D13.2 (A), U7.2 (DESAT)
- new net: R26.1, U7.4 (OUTH)
- new net: R27.2, U7.6 (OUTL)
- new net: J17.2 (Pin_2), U7.8 (VEE2)
- new net: R33.2, U8.6 (OUTL)
- new net: D13.1 (K), R25.2
- new net: J15.2 (Pin_2), U5.8 (VEE2)
- new net: R18.2, U5.6 (OUTL)
- new net: J18.2 (Pin_2), U8.8 (VEE2)
- new net: D11.1 (K), R19.2
- new net: D11.2 (A), U6.2 (DESAT)
- new net: D10.1 (K), R16.2
- new net: D10.2 (A), U5.2 (DESAT)
- new net: R17.1, U5.4 (OUTH)
- new net: R20.1, U6.4 (OUTH)
- new net: R21.2, U6.6 (OUTL)
- new net: J16.2 (Pin_2), U6.8 (VEE2)
- new net: R32.1, U8.4 (OUTH)
- new net +15_DRV2: C2.2, C4.2, C5.2, C6.2, J12.1 (Pin_1), J3.1 (Pin_1), J6.1 (Pin_1), J9.1 (Pin_1), U5.5 (VCC2), U6.5 (VCC2), U7.5 (VCC2), U8.5 (VCC2)
- new net +3V3_DRV1: C1.1, J1.6 (Pin_6), J10.6 (Pin_6), J14.1 (Pin_1), J4.6 (Pin_6), J7.6 (Pin_6), R13.1, R14.1, R15.1, R22.1, R23.1, R24.1, R28.1, R29.1, R30.1, R34.1, R35.1, R36.1, U1.3 (OUT), U5.15 (VCC1), U6.15 (VCC1), U7.15 (VCC1), U8.15 (VCC1)
- new net -15_DRV2: J12.3 (Pin_3), J15.3 (Pin_3), J16.3 (Pin_3), J17.3 (Pin_3), J18.3 (Pin_3), J3.3 (Pin_3), J6.3 (Pin_3), J9.3 (Pin_3)
- new net EN1: J1.5 (Pin_5), R13.2, U5.14 (~{RST}/EN)
- new net EN2: J4.5 (Pin_5), R22.2, U6.14 (~{RST}/EN)
- new net EN3: J7.5 (Pin_5), R28.2, U7.14 (~{RST}/EN)
- new net EN4: J10.5 (Pin_5), R34.2, U8.14 (~{RST}/EN)
- new net FLT1: D8.1 (K), J1.4 (Pin_4), R14.2, U5.13 (~{FLT})
- new net FLT2: D9.1 (K), J4.4 (Pin_4), R23.2, U6.13 (~{FLT})
- new net FLT3: D14.1 (K), J7.4 (Pin_4), R29.2, U7.13 (~{FLT})
- new net FLT4: D17.1 (K), J10.4 (Pin_4), R35.2, U8.13 (~{FLT})
- new net GND_DRV1: C1.2, C3.2, D12.2 (A), D14.2 (A), D15.2 (A), D17.2 (A), D18.2 (A), D7.2 (A), D8.2 (A), D9.2 (A), J1.1 (Pin_1), J10.1 (Pin_1), J4.1 (Pin_1), J7.1 (Pin_1), U1.2 (GND), U5.11 (IN-), U5.9 (GND1), U6.11 (IN-), U6.9 (GND1), U7.11 (IN-), U7.9 (GND1), U8.11 (IN-), U8.9 (GND1)
- new net GND_DRV2: C2.1, C4.1, C5.1, C6.1, J11.3 (Pin_3), J12.2 (Pin_2), J15.1 (Pin_1), J16.1 (Pin_1), J17.1 (Pin_1), J18.1 (Pin_1), J2.3 (Pin_3), J3.2 (Pin_2), J5.3 (Pin_3), J6.2 (Pin_2), J8.3 (Pin_3), J9.2 (Pin_2), Q1.3 (S), Q2.3 (S), Q3.3 (S), Q4.3 (S), TP11.1, TP3.1, TP5.1, TP8.1, U5.3 (GND2), U6.3 (GND2), U7.3 (GND2), U8.3 (GND2)
- new net IN1: J1.2 (Pin_2), U5.10 (IN+)
- new net IN2: J4.2 (Pin_2), U6.10 (IN+)
- new net IN3: J7.2 (Pin_2), U7.10 (IN+)
- new net IN4: J10.2 (Pin_2), U8.10 (IN+)
- new net RDY1: D7.1 (K), J1.3 (Pin_3), R15.2, U5.12 (RDY)
- new net RDY2: D12.1 (K), J4.3 (Pin_3), R24.2, U6.12 (RDY)
- new net RDY3: D15.1 (K), J7.3 (Pin_3), R30.2, U7.12 (RDY)
- new net RDY4: D18.1 (K), J10.3 (Pin_3), R36.2, U8.12 (RDY)
- new net drain1: J2.2 (Pin_2), Q1.2 (D), R16.1, TP2.1
- new net drain2: J5.2 (Pin_2), Q2.2 (D), R19.1, TP4.1
- new net drain3: J8.2 (Pin_2), Q3.2 (D), R25.1, TP7.1
- new net drain4: J11.2 (Pin_2), Q4.2 (D), R31.1, TP10.1
- new net gate1: J2.1 (Pin_1), Q1.1 (G), R17.2, R18.1, TP1.1, U5.7 (CLAMP)
- new net gate2: J5.1 (Pin_1), Q2.1 (G), R20.2, R21.1, TP6.1, U6.7 (CLAMP)
- new net gate3: J8.1 (Pin_1), Q3.1 (G), R26.2, R27.1, TP9.1, U7.7 (CLAMP)
- new net gate4: J11.1 (Pin_1), Q4.1 (G), R32.2, R33.1, TP12.1, U8.7 (CLAMP)
- no-connect marks 0 -> 8
