File: hbridge/logic_defence.kicad_sch (KiCad schematic)
At the start: 8 parts, among them J23 Conn_01x03, J24 Conn_01x08_Pin, SW1 SW_Push, U10 74HC165, U13 CD4043B, U6 MC74HC08ADG (74HC08), U8 74AHC04

Commit message: Half-bridge refactoring start.
Parts:
- R20: footprint (none) -> Resistor_SMD:R_0805_2012Metric_Pad1.20x1.40mm_HandSolder
- U13: footprint (none) -> Package_SO:SOIC-16_3.9x9.9mm_P1.27mm
- U13: footprint Package_SO:SOIC-14_3.9x8.7mm_P1.27mm -> Package_SO:SOIC-16_3.9x9.9mm_P1.27mm
Changed lines of the file:
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@@
 			)
 		)
-		(property "Footprint" ""
+		(property "Footprint" "Package_SO:SOIC-16_3.9x9.9mm_P1.27mm"
 			(at 181.61 41.91 0)
 			(hide yes)
@@
 			)
 		)
-		(property "Datasheet" "https://www.ti.com/lit/gpn/sn54ls279a"
+		(property "Datasheet" "https://static.chipdip.ru/lib/947/DOC005947915.pdf"
 			(at 192.532 54.864 0)
 			(hide yes)
@@
 			)
 		)
-		(property "Footprint" ""
+		(property "Footprint" "Package_SO:SOIC-16_3.9x9.9mm_P1.27mm"
 			(at 181.61 95.25 0)
 			(hide yes)
@@
 			)
 		)
-		(property "Datasheet" "https://www.ti.com/lit/gpn/sn54ls279a"
+		(property "Datasheet" "https://static.chipdip.ru/lib/947/DOC005947915.pdf"
 			(at 192.532 108.204 0)
 			(hide yes)
@@
 			)
 		)
-		(property "Footprint" ""
+		(property "Footprint" "Package_SO:SOIC-16_3.9x9.9mm_P1.27mm"
 			(at 181.61 59.69 0)
 			(hide yes)
@@
 			)
 		)
-		(property "Datasheet" "https://www.ti.com/lit/gpn/sn54ls279a"
+		(property "Datasheet" "https://static.chipdip.ru/lib/947/DOC005947915.pdf"
 			(at 192.532 72.644 0)
 			(hide yes)
@@
 			)
 		)
-		(property "Footprint" "Package_SO:SOIC-14_3.9x8.7mm_P1.27mm"
+		(property "Footprint" "Package_SO:SOIC-16_3.9x9.9mm_P1.27mm"
 			(at 105.41 167.64 0)
 			(hide yes)
@@
 			)
 		)
-		(property "Footprint" ""
+		(property "Footprint" "Package_SO:SOIC-16_3.9x9.9mm_P1.27mm"
 			(at 181.61 77.47 0)
 			(hide yes)
@@
 			)
 		)
-		(property "Datasheet" "https://www.ti.com/lit/gpn/sn54ls279a"
+		(property "Datasheet" "https://static.chipdip.ru/lib/947/DOC005947915.pdf"
 			(at 192.532 90.424 0)
 			(hide yes)
@@
 			)
 		)
-		(property "Footprint" ""
+		(property "Footprint" "Resistor_SMD:R_0805_2012Metric_Pad1.20x1.40mm_HandSolder"
 			(at 155.702 106.68 90)
 			(hide yes)
