File: ierarchy_schematics/drv_opt.kicad_sch (KiCad schematic)
At the start: 11 parts, among them J20 to_mcu_opt, J22 to_driver_opt, U5 Optocoupler_4chan

Commit message: Lab consultation.
Other:
- note added: "питание 12в у драйвера свое hlk маленький"
- note added: "сделать защиту от сжигания полумоста. передавать управление на мк. учесть то, что переменное напряжение"
Changed lines of the file:
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@@
 	(generator_version "10.0")
 	(paper "A4")
+	(text "питание 12в у драйвера свое\nhlk маленький"
+		(exclude_from_sim no)
+		(at 233.426 58.928 0)
+		(effects
+			(font
+				(size 1.27 1.27)
+			)
+		)
+	)
+	(text "сделать защиту от сжигания полумоста. передавать управление на мк.\nучесть то, что переменное напряжение"
+		(exclude_from_sim no)
+		(at 237.49 105.41 0)
+		(effects
+			(font
+				(size 1.27 1.27)
+			)
+		)
+	)
 	(text "подтяжка к 3.3В на плате драйвера"
 		(exclude_from_sim no)
