File: ierarchy_schematics/hbr_power.kicad_sch (KiCad schematic)
At the start: 10 parts, among them J17 Conn_01x01_Socket, J18 Conn_01x01_Socket, J19 24V, U1 LDO-3.3, U10 AM6TW-2415DZ, U20 B2412S-2WR3, U4 AM6TW-2415DZ

Commit message: Lab consultation.
Parts:
- added C5, C8: C, Capacitor_SMD:C_0805_2012Metric_Pad1.18x1.45mm_HandSolder, symbol Device:C
- added J21: Conn_01x01_Socket, TestPoint:TestPoint_Loop_D1.80mm_Drill1.0mm_Beaded, symbol Connector:Conn_01x01_Socket
- added U21: B2412S-2WR3, TerminalBlock:TerminalBlock_Xinya_XY308-2.54-6P_1x06_P2.54mm_Horizontal, symbol Regulator_Linear:LDK130-ADJ_DFN6
- added U8: LDO-12, Package_TO_SOT_SMD:SOT-223-3_TabPin2, symbol Regulator_Linear:LT1963AxST-3.3
Connections:
- net +12V: now also C5.1, J21.1 (Pin_1), U21.6 (+VOUT), U8.3 (OUT)
- net +24V_1: now also U21.1 (VIN)
- net GND1: now also U21.2 (GND_IN)
- net GND_DRV1: now also C5.2, C8.2, U21.4 (GND_OUT), U8.2 (GND)
- new net +12: C8.1, U8.1 (IN)
Other:
- note added: "24V берем от HIGH, LOW силы + выпрямитель диодный мост от 9 до 36 В +LC фильтр сравнить диодный мост с корректором SDH7711"
- note added: "proteus, orcad"
