File: mcu_board/mcu_board.kicad_pcb (KiCad board)
At the start: 2 copper layers, 1 part, among them U1 STM32G474_LQFP48(chip)

Commit message: Library updated and other changes.
Parts:
- added U2: HLK-40M24, Converter_ACDC:Converter_ACDC_Hi-Link_HLK-30Mxx, F.Cu at (46.0, 79.3)
Changed lines of the file:
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@@
+		)
+	)
+	(footprint "Converter_ACDC:Converter_ACDC_Hi-Link_HLK-30Mxx"
+		(layer "F.Cu")
+		(at 46.03 79.335)
+		(descr "ACDC-Converter, 30W, Hi-Link, HLK-30Mxx, HLK-30MxxC, THT, https://h.hlktech.com/download/ACDC%E7%94%B5%E6%BA%90%E6%A8%A1%E5%9D%9730W%E7%B3%BB%E5%88%97/1/%E6%B5%B7%E5%87%8C%E7%A7%9130W%E7%B3%BB%E5%88%97%E7%94%B5%E6%BA%90%E6%A8%A1%E5%9D%97%E8%A7%84%E6%A0%BC%E4%B9%A6V1.6.pdf")
+		(tags "ACDC-Converter 30W THT Hi-Link board mount module")
+		(property "Reference" "U2"
+			(at 25.5 -22.51 0)
+			(layer "F.SilkS")
+			(effects
+				(font
+					(size 1 1)
+					(thickness 0.15)
+				)
+			)
+		)
+		(property "Value" "HLK-40M24"
+			(at 25.5 14.89 0)
+			(layer "F.Fab")
+			(effects
+				(font
+					(size 1 1)
+					(thickness 0.15)
+				)
+			)
+		)
+		(property "Datasheet" ""
+			(at 0 0 0)
+			(layer "F.Fab")
+			(hide yes)
+			(effects
+				(font
+					(size 1.27 1.27)
+				)
+			)
+		)
+		(property "Description" "Compact AC/DC board mount power module 20W 5V"
+			(at 0 0 0)
+			(layer "F.Fab")
+			(hide yes)
+			(effects
+				(font
+					(size 1.27 1.27)
+				)
+			)
+		)
+		(property "KiLib_Generator" "converter_ACDC_DCDC"
+			(at 0 0 0)
+			(layer "F.SilkS")
+			(hide yes)
+			(effects
+				(font
+					(size 1 1)
+					(thickness 0.15)
+				)
+			)
+		)
+		(property ki_fp_filters "Converter*ACDC*Hi?Link*HLK?20M*")
+		(sheetname "/")
+		(sheetfile "mcu_board.kicad_sch")
+		(units
+			(unit
+				(name "A")
+				(pins "1" "2" "6" "3")
+			)
+		)
+		(attr through_hole)
+		(duplicate_pad_numbers_are_jumpers no)
+		(fp_line
+			(start -4.36 -21.67)
+			(end 55.36 -21.67)
+			(stroke
+				(width 0.12)
+				(type solid)
+			)
+			(layer "F.SilkS")
+		)
+		(fp_line
+			(start -4.36 -0.296)
+			(end -4.36 -21.67)
+			(stroke
+				(width 0.12)
+				(type solid)
+			)
+			(layer "F.SilkS")
+		)
+		(fp_line
+			(start -4.36 14.05)
+			(end -4.36 0.296)
+			(stroke
+				(width 0.12)
+				(type solid)
+			)
+			(layer "F.SilkS")
+		)
+		(fp_line
+			(start 55.36 -21.67)
+			(end 55.36 14.05)
+			(stroke
+				(width 0.12)
+				(type solid)
+			)
+			(layer "F.SilkS")
+		)
+		(fp_line
+			(start 55.36 14.05)
+			(end -4.36 14.05)
+			(stroke
+				(width 0.12)
+				(type solid)
+			)
+			(layer "F.SilkS")
+		)
+		(fp_poly
+			(pts
+				(xy -4.36 0) (xy -4.97 0.44) (xy -4.97 -0.44)
+			)
+			(stroke
+				(width 0.12)
+				(type solid)
+			)
+			(fill yes)
+			(layer "F.SilkS")
+		)
+		(fp_rect
+			(start -4.5 -21.81)
+			(end 55.5 14.19)
+			(stroke
+				(width 0.05)
+				(type solid)
+			)
+			(fill no)
+			(layer "F.CrtYd")
+		)
+		(fp_poly
+			(pts
+				(xy -2.25 -20.56) (xy 54.25 -20.56) (xy 54.25 12.94) (xy -3.25 12.94) (xy -3.25 -19.56)
+			)
+			(stroke
+				(width 0.1)
+				(type solid)
+			)
+			(fill no)
+			(layer "F.Fab")
+		)
+		(fp_text user "${REFERENCE}"
+			(at 25.5 -3.81 0)
+			(layer "F.Fab")
+			(effects
+				(font
+					(size 1 1)
+					(thickness 0.15)
+				)
+			)
+		)
+		(pad "1" thru_hole roundrect
+			(at 0 0)
+			(size 2 2.3)
+			(drill 1.3)
+			(layers "*.Cu" "*.Mask")
+			(remove_unused_layers no)
+			(roundrect_rratio 0.125)
+			(net "unconnected-(U2-AC{slash}L-Pad1)")
+			(pinfunction "AC/L_1")
+			(pintype "power_in")
+		)
+		(pad "2" thru_hole oval
+			(at 0 5.08)
+			(size 2 2.3)
+			(drill 1.3)
+			(layers "*.Cu" "*.Mask")
+			(remove_unused_layers no)
+			(net "unconnected-(U2-AC{slash}N-Pad2)")
+			(pinfunction "AC/N_2")
+			(pintype "power_in")
+		)
+		(pad "3" thru_hole oval
+			(at 51 -17.78)
+			(size 2 2.3)
+			(drill 1.3)
+			(layers "*.Cu" "*.Mask")
+			(remove_unused_layers no)
+			(net "unconnected-(U2--Vout-Pad3)")
+			(pinfunction "-Vout_3")
+			(pintype "power_out")
+		)
+		(pad "6" thru_hole oval
+			(at 51 -10.16)
+			(size 2 2.3)
+			(drill 1.3)
+			(layers "*.Cu" "*.Mask")
+			(remove_unused_layers no)
+			(net "unconnected-(U2-+Vout-Pad6)")
+			(pinfunction "+Vout_6")
+			(pintype "power_out")
+		)
+		(embedded_fonts no)
+		(model "${KICAD10_3DMODEL_DIR}/Converter_ACDC.3dshapes/Converter_ACDC_Hi-Link_HLK-30Mxx.step"
+			(offset
+				(xyz 0 0 0)
+			)
+			(scale
+				(xyz 1 1 1)
+			)
+			(rotate
+				(xyz 0 0 0)
+			)
 		)
 	)
