File: mcu_board/mcu_board.kicad_sch (KiCad schematic)
At the start: 1 part, among them U1 STM32G474_LQFP48(chip)

Commit message: Library updated and other changes.
Parts:
- added U2: HLK-40M24, Converter_ACDC:Converter_ACDC_Hi-Link_HLK-30Mxx, symbol Converter_ACDC:HLK-20M05
Other:
- moved on the sheet: U1
Changed lines of the file:
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@@
 	(symbol
 		(lib_id "Tamara:STM32G474_WeAct_Long")
-		(at 200.66 85.09 0)
+		(at 201.93 53.34 0)
 		(unit 1)
 		(body_style 1)
@@
 		(fields_autoplaced yes)
 		(property "Reference" "U1"
-			(at 201.295 62.23 0)
+			(at 202.565 30.48 0)
 			(show_name no)
 			(do_not_autoplace no)
@@
 		)
 		(property "Value" "STM32G474_LQFP48(chip)"
-			(at 201.295 64.77 0)
+			(at 202.565 33.02 0)
 			(show_name no)
 			(do_not_autoplace no)
@@
 		)
 		(property "Footprint" "Package_DIP:DIP-48_W15.24mm_LongPads"
-			(at 283.21 129.54 0)
+			(at 284.48 97.79 0)
 			(hide yes)
 			(show_name no)
@@
 		)
 		(property "Datasheet" ""
-			(at 185.928 58.42 0)
+			(at 187.198 26.67 0)
 			(hide yes)
 			(show_name no)
@@
 		)
 		(property "Description" "High and Low Side Gate Driver, 200V operation, Output Current 350/650mA, SOIC-8"
-			(at 167.386 63.246 0)
+			(at 168.656 31.496 0)
 			(hide yes)
 			(show_name no)
@@
 					(unit 1)
 				)
+			)
+		)
+	)
+	(symbol
+		(lib_id "Converter_ACDC:HLK-20M05")
+		(at 40.64 45.72 0)
+		(unit 1)
+		(body_style 1)
+		(exclude_from_sim no)
+		(in_bom yes)
+		(on_board yes)
+		(in_pos_files yes)
+		(dnp no)
+		(fields_autoplaced yes)
+		(property "Reference" "U2"
+			(at 40.64 36.83 0)
+			(show_name no)
+			(do_not_autoplace no)
+			(effects
+				(font
+					(size 1.27 1.27)
+				)
+			)
+		)
+		(property "Value" "HLK-40M24"
+			(at 40.64 39.37 0)
+			(show_name no)
+			(do_not_autoplace no)
+			(effects
+				(font
+					(size 1.27 1.27)
+				)
+			)
+		)
+		(property "Footprint" "Converter_ACDC:Converter_ACDC_Hi-Link_HLK-30Mxx"
+			(at 40.64 52.705 0)
+			(hide yes)
+			(show_name no)
+			(do_not_autoplace no)
+			(effects
+				(font
+					(size 1.27 1.27)
+				)
+			)
+		)
+		(property "Datasheet" ""
+			(at 40.64 54.61 0)
+			(hide yes)
+			(show_name no)
+			(do_not_autoplace no)
+			(effects
+				(font
+					(size 1.27 1.27)
+				)
+			)
+		)
+		(property "Description" "Compact AC/DC board mount power module 20W 5V"
+			(at 40.64 45.72 0)
+			(hide yes)
+			(show_name no)
+			(do_not_autoplace no)
+			(effects
+				(font
+					(size 1.27 1.27)
+				)
+			)
+		)
+		(pin "3"
+		)
+		(pin "1"
+		)
+		(pin "2"
+		)
+		(pin "6"
+		)
+		(instances
+			(project "mcu_board"
+				(path "/6c7a03e4-c8d1-47f7-b15e-d483cc6a10af"
+					(reference "U2")
+					(unit 1)
+				)
